File: 0-10v_PCB/pwm_0-10v/untitled.brd (EAGLE design)
At the start: 160 x 100 mm, 5 parts, among them U1 OP07CDR, X1 MKDSN1,5/2-5,08, X2 MKDSN1,5/2-5,08

Commit message: made .brd file
Parts:
- removed R2: 10k, rcl:R0805
- removed X1, X2: MKDSN1,5/2-5,08, con-phoenix-508:MKDSN1,5/2-5,08
- added R1: 10k, rcl:M0805
- added SL1, SL2: (no value), con-amp-quick:02P
- moved U1 21.7 mm to (6.35, 6.35)
- moved C1 13.1 mm to (8.89, 21.6), turned to 0 degrees
Connections:
- net +12V: now also SL2.1; no longer X2.1
- net GND: now also SL2.2; no longer X2.2
- net N$1: now also R1.1, SL1.1; no longer C1.1, R2.2, U1.3
- net N$2: now also C1.1, R1.2, U1.3; no longer X1.2
- net N$3: now also SL1.2; no longer R2.1, X1.1
Changed lines of the file:
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@@
 </autorouter>
 <elements>
-<element name="U1" library="OP07CDR" package="SOIC127P599X175-8N" value="OP07CDR" x="8.89" y="27.94" smashed="yes">
-<attribute name="AVAILABILITY" value="Warning" x="27.94" y="-10.16" size="1.778" layer="27" display="off"/>
-<attribute name="DESCRIPTION" value=" Low-Offset voltage (0.25mV) single operational amplifier 8-SOIC 0 to 70 " x="27.94" y="-10.16" size="1.778" layer="27" display="off"/>
-<attribute name="MF" value="Texas Instruments" x="27.94" y="-10.16" size="1.778" layer="27" display="off"/>
-<attribute name="MP" value="OP07CDR" x="27.94" y="-10.16" size="1.778" layer="27" display="off"/>
-<attribute name="NAME" x="5.33" y="30.842" size="1.27" layer="25"/>
-<attribute name="PACKAGE" value="SOIC-8 Texas Instruments" x="27.94" y="-10.16" size="1.778" layer="27" display="off"/>
-<attribute name="PRICE" value="None" x="27.94" y="-10.16" size="1.778" layer="27" display="off"/>
-<attribute name="PURCHASE-URL" value="https://pricing.snapeda.com/search/part/OP07CDR/?ref=eda" x="27.94" y="-10.16" size="1.778" layer="27" display="off"/>
-<attribute name="VALUE" x="5.33" y="25.038" size="1.27" layer="27" align="top-left"/>
+<element name="C1" library="rcl" library_urn="urn:adsk.eagle:library:334" package="C0805" package3d_urn="urn:adsk.eagle:package:23617/2" value="10uF" x="8.89" y="21.59" smashed="yes">
+<attribute name="NAME" x="7.62" y="22.86" size="1.27" layer="25"/>
+<attribute name="POPULARITY" value="88" x="25.4" y="0" size="1.778" layer="27" display="off"/>
+<attribute name="SPICEPREFIX" value="C" x="25.4" y="0" size="1.778" layer="27" display="off"/>
+<attribute name="VALUE" x="7.62" y="19.05" size="1.27" layer="27"/>
 </element>
-<element name="X1" library="con-phoenix-508" library_urn="urn:adsk.eagle:library:176" package="MKDSN1,5/2-5,08" package3d_urn="urn:adsk.eagle:package:9630/1" value="MKDSN1,5/2-5,08" x="7.62" y="16.51" smashed="yes">
-<attribute name="NAME" x="2.8689" y="20.955" size="1.27" layer="25"/>
-<attribute name="POPULARITY" value="14" x="27.94" y="11.43" size="1.778" layer="27" display="off"/>
-<attribute name="VALUE" x="14.605" y="12.7" size="1.27" layer="27" rot="R90"/>
+<element name="R1" library="rcl" library_urn="urn:adsk.eagle:library:334" package="M0805" package3d_urn="urn:adsk.eagle:package:23556/2" value="10k" x="3.81" y="21.59" smashed="yes">
+<attribute name="NAME" x="2.54" y="22.86" size="1.27" layer="25"/>
+<attribute name="POPULARITY" value="45" x="25.4" y="0" size="1.778" layer="27" display="off"/>
+<attribute name="SPICEPREFIX" value="R" x="25.4" y="0" size="1.778" layer="27" display="off"/>
+<attribute name="VALUE" x="2.54" y="19.05" size="1.27" layer="27"/>
 </element>
-<element name="X2" library="con-phoenix-508" library_urn="urn:adsk.eagle:library:176" package="MKDSN1,5/2-5,08" package3d_urn="urn:adsk.eagle:package:9630/1" value="MKDSN1,5/2-5,08" x="8.89" y="41.91" smashed="yes">
-<attribute name="NAME" x="4.1389" y="46.355" size="1.27" layer="25"/>
-<attribute name="POPULARITY" value="14" x="29.21" y="20.32" size="1.778" layer="27" display="off"/>
-<attribute name="VALUE" x="15.875" y="38.1" size="1.27" layer="27" rot="R90"/>
+<element name="SL1" library="con-amp-quick" library_urn="urn:adsk.eagle:library:125" package="02P" package3d_urn="urn:adsk.eagle:package:5956/1" value="" x="10.16" y="12.7" smashed="yes">
+<attribute name="MF" value="" x="25.4" y="0" size="1.778" layer="27" display="off"/>
+<attribute name="MPN" value="" x="25.4" y="0" size="1.778" layer="27" display="off"/>
+<attribute name="NAME" x="7.874" y="15.6464" size="1.27" layer="25" ratio="10"/>
+<attribute name="OC_FARNELL" value="unknown" x="25.4" y="0" size="1.778" layer="27" display="off"/>
+<attribute name="OC_NEWARK" value="unknown" x="25.4" y="0" size="1.778" layer="27" display="off"/>
+<attribute name="POPULARITY" value="33" x="25.4" y="0" size="1.778" layer="27" display="off"/>
+<attribute name="VALUE" x="7.874" y="8.8646" size="1.27" layer="27" ratio="10"/>
 </element>
-<element name="C1" library="rcl" library_urn="urn:adsk.eagle:library:334" package="C0805" package3d_urn="urn:adsk.eagle:package:23617/2" value="10uF" x="2.54" y="33.02" smashed="yes" rot="R90">
-<attribute name="NAME" x="1.27" y="31.75" size="1.27" layer="25" rot="R90"/>
-<attribute name="POPULARITY" value="88" x="2.54" y="33.02" size="1.778" layer="27" rot="R90" display="off"/>
-<attribute name="SPICEPREFIX" value="C" x="2.54" y="33.02" size="1.778" layer="27" rot="R90" display="off"/>
-<attribute name="VALUE" x="5.08" y="31.75" size="1.27" layer="27" rot="R90"/>
+<element name="SL2" library="con-amp-quick" library_urn="urn:adsk.eagle:library:125" package="02P" package3d_urn="urn:adsk.eagle:package:5956/1" value="" x="3.81" y="12.7" smashed="yes">
+<attribute name="MF" value="" x="25.4" y="0" size="1.778" layer="27" display="off"/>
+<attribute name="MPN" value="" x="25.4" y="0" size="1.778" layer="27" display="off"/>
+<attribute name="NAME" x="1.524" y="15.6464" size="1.27" layer="25" ratio="10"/>
+<attribute name="OC_FARNELL" value="unknown" x="25.4" y="0" size="1.778" layer="27" display="off"/>
+<attribute name="OC_NEWARK" value="unknown" x="25.4" y="0" size="1.778" layer="27" display="off"/>
+<attribute name="POPULARITY" value="33" x="25.4" y="0" size="1.778" layer="27" display="off"/>
+<attribute name="VALUE" x="1.524" y="8.8646" size="1.27" layer="27" ratio="10"/>
 </element>
-<element name="R2" library="rcl" library_urn="urn:adsk.eagle:library:334" package="R0805" package3d_urn="urn:adsk.eagle:package:23553/2" value="10k" x="2.54" y="27.94" smashed="yes" rot="R90">
-<attribute name="NAME" x="1.27" y="27.305" size="1.27" layer="25" rot="R90"/>
-<attribute name="POPULARITY" value="86" x="2.54" y="27.94" size="1.778" layer="27" rot="R90" display="off"/>
-<attribute name="SPICEPREFIX" value="R" x="2.54" y="27.94" size="1.778" layer="27" rot="R90" display="off"/>
-<attribute name="VALUE" x="5.08" y="27.305" size="1.27" layer="27" rot="R90"/>
+<element name="U1" library="OP07CDR" package="SOIC127P599X175-8N" value="OP07CDR" x="6.35" y="6.35" smashed="yes">
+<attribute name="AVAILABILITY" value="Warning" x="25.4" y="1.27" size="1.778" layer="27" display="off"/>
+<attribute name="DESCRIPTION" value=" Low-Offset voltage (0.25mV) single operational amplifier 8-SOIC 0 to 70 " x="25.4" y="1.27" size="1.778" layer="27" display="off"/>
+<attribute name="MF" value="Texas Instruments" x="25.4" y="1.27" size="1.778" layer="27" display="off"/>
+<attribute name="MP" value="OP07CDR" x="25.4" y="1.27" size="1.778" layer="27" display="off"/>
+<attribute name="NAME" x="2.79" y="9.252" size="1.27" layer="25"/>
+<attribute name="PACKAGE" value="SOIC-8 Texas Instruments" x="25.4" y="1.27" size="1.778" layer="27" display="off"/>
+<attribute name="PRICE" value="None" x="25.4" y="1.27" size="1.778" layer="27" display="off"/>
+<attribute name="PURCHASE-URL" value="https://pricing.snapeda.com/search/part/OP07CDR/?ref=eda" x="25.4" y="1.27" size="1.778" layer="27" display="off"/>
+<attribute name="VALUE" x="2.79" y="3.448" size="1.27" layer="27" align="top-left"/>
 </element>
 </elements>
 <signals>
 <signal name="GND">
+<contactref element="SL2" pad="2"/>
 <contactref element="U1" pad="4"/>
-<contactref element="X2" pad="2"/>
 <contactref element="C1" pad="2"/>
-<wire x1="11.4089" y1="41.935" x2="2.54" y2="33.97" width="0" layer="19" extent="1-1"/>
-<wire x1="6.42" y1="26.035" x2="11.4089" y2="41.935" width="0" layer="19" extent="1-1"/>
+<wire x1="5.08" y1="12.7" x2="3.88" y2="4.445" width="0" layer="19" extent="1-1"/>
+<wire x1="9.84" y1="21.59" x2="5.08" y2="12.7" width="0" layer="19" extent="1-1"/>
 </signal>
 <signal name="+12V">
-<contactref element="X2" pad="1"/>
+<contactref element="SL2" pad="1"/>
 <contactref element="U1" pad="7"/>
-<wire x1="6.3289" y1="41.935" x2="11.36" y2="28.575" width="0" layer="19" extent="1-1"/>
+<wire x1="8.82" y1="6.985" x2="2.54" y2="12.7" width="0" layer="19" extent="1-1"/>
+</signal>
+<signal name="N$1">
+<contactref element="SL1" pad="1"/>
+<contactref element="R1" pad="1"/>
+<wire x1="2.86" y1="21.59" x2="8.89" y2="12.7" width="0" layer="19" extent="1-1"/>
+</signal>
+<signal name="N$2">
+<contactref element="R1" pad="2"/>
+<contactref element="U1" pad="3"/>
+<contactref element="C1" pad="1"/>
+<wire x1="4.76" y1="21.59" x2="3.88" y2="5.715" width="0" layer="19" extent="1-1"/>
+<wire x1="7.94" y1="21.59" x2="4.76" y2="21.59" width="0" layer="19" extent="1-1"/>
 </signal>
 <signal name="OUT_A">
 <contactref element="U1" pad="2"/>
 <contactref element="U1" pad="6"/>
-<wire x1="6.42" y1="28.575" x2="11.36" y2="27.305" width="0" layer="19" extent="1-1"/>
-</signal>
-<signal name="N$2">
-<contactref element="X1" pad="2"/>
-</signal>
-<signal name="N$1">
-<contactref element="U1" pad="3"/>
-<contactref element="C1" pad="1"/>
-<contactref element="R2" pad="2"/>
-<wire x1="2.54" y1="32.07" x2="2.54" y2="28.89" width="0" layer="19" extent="1-1"/>
-<wire x1="6.42" y1="27.305" x2="2.54" y2="32.07" width="0" layer="19" extent="1-1"/>
+<wire x1="8.82" y1="5.715" x2="3.88" y2="6.985" width="0" layer="19" extent="1-1"/>
 </signal>
 <signal name="N$3">
-<contactref element="X1" pad="1"/>
-<contactref element="R2" pad="1"/>
-<wire x1="5.0589" y1="16.535" x2="2.54" y2="26.99" width="0" layer="19" extent="1-1"/>
+<contactref element="SL1" pad="2"/>
 </signal>
 </signals>
