File: 0-10v_PCB/pwm_0-10v/untitled.brd (EAGLE design)
At the start: 51.5 x 28.2 mm, 16 parts, among them U1 OP07CDR, U2 OP07CDR, U3 OP07CDR

Commit message: changed pulldown resistors to 1.5k instead of 10k
Parts:
- R4, R5, R6: value 10k -> 1.5k
Changed lines of the file:
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@@
 <attribute name="VALUE" x="28.575" y="15.875" size="1.778" layer="27" ratio="10" rot="R90"/>
 </element>
-<element name="R4" library="rcl" library_urn="urn:adsk.eagle:library:334" package="M0805" package3d_urn="urn:adsk.eagle:package:23556/2" value="10k" x="-1.905" y="25.4" smashed="yes" rot="R90">
+<element name="R4" library="rcl" library_urn="urn:adsk.eagle:library:334" package="M0805" package3d_urn="urn:adsk.eagle:package:23556/2" value="1.5k" x="-1.905" y="25.4" smashed="yes" rot="R90">
 <attribute name="NAME" x="-3.175" y="24.13" size="1.27" layer="25" rot="R90"/>
 <attribute name="POPULARITY" value="45" x="-1.905" y="25.4" size="1.778" layer="27" rot="R90" display="off"/>
@@
 <attribute name="VALUE" x="0.635" y="24.13" size="1.27" layer="27" rot="R90"/>
 </element>
-<element name="R5" library="rcl" library_urn="urn:adsk.eagle:library:334" package="M0805" package3d_urn="urn:adsk.eagle:package:23556/2" value="10k" x="-10.795" y="25.4" smashed="yes" rot="R90">
+<element name="R5" library="rcl" library_urn="urn:adsk.eagle:library:334" package="M0805" package3d_urn="urn:adsk.eagle:package:23556/2" value="1.5k" x="-10.795" y="25.4" smashed="yes" rot="R90">
 <attribute name="NAME" x="-12.065" y="24.13" size="1.27" layer="25" rot="R90"/>
 <attribute name="POPULARITY" value="45" x="-10.795" y="25.4" size="1.778" layer="27" rot="R90" display="off"/>
@@
 <attribute name="VALUE" x="-8.255" y="24.13" size="1.27" layer="27" rot="R90"/>
 </element>
-<element name="R6" library="rcl" library_urn="urn:adsk.eagle:library:334" package="M0805" package3d_urn="urn:adsk.eagle:package:23556/2" value="10k" x="6.985" y="25.4" smashed="yes" rot="R90">
+<element name="R6" library="rcl" library_urn="urn:adsk.eagle:library:334" package="M0805" package3d_urn="urn:adsk.eagle:package:23556/2" value="1.5k" x="6.985" y="25.4" smashed="yes" rot="R90">
 <attribute name="NAME" x="5.715" y="24.13" size="1.27" layer="25" rot="R90"/>
 <attribute name="POPULARITY" value="45" x="6.985" y="25.4" size="1.778" layer="27" rot="R90" display="off"/>
